File: pcb/RS485.kicad_sch (KiCad schematic)
At the start: 5 parts, among them U8 THVD1400D

Commit message: Swap 1Wire and AC sense
Parts:
- C24: LCSC (none) -> C1525
- D5: LCSC (none) -> C172881
- U8: LCSC (none) -> C3235232
Changed lines of the file:
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@@
+      (effects (font (size 1.27 1.27)) hide)
+    )
+    (property "LCSC" "C1525" (at 156.21 139.7 0)
       (effects (font (size 1.27 1.27)) hide)
     )
@@
     )
     (property "Datasheet" "https://www.ti.com/lit/ds/symlink/thvd1420.pdf" (at 156.21 93.98 0)
+      (effects (font (size 1.27 1.27)) hide)
+    )
+    (property "LCSC" "C3235232" (at 156.21 95.25 0)
       (effects (font (size 1.27 1.27)) hide)
     )
@@
       (effects (font (size 1.27 1.27)) hide)
     )
+    (property "LCSC" "C172881" (at 121.92 110.49 0)
+      (effects (font (size 1.27 1.27)) hide)
+    )
