File: pcb/boost.kicad_sch (KiCad schematic)
At the start: 10 parts

Commit message: Swap 1Wire and AC sense
Parts:
- added TP3: TestPoint, TestPoint:TestPoint_Pad_D1.0mm, symbol Connector:TestPoint
- C?: LCSC (none) -> C1683
- C? (x3): LCSC (none) -> C23630
- D?: value MBR0550 -> MBR0580; LCSC (none) -> C177047
- L?: LCSC (none) -> C2045998
- R?: LCSC (none) -> C122547
- R?: value 47K -> 100K; LCSC (none) -> C25741
- R?: LCSC (none) -> C25557
- U?: LCSC (none) -> C78226
Connections:
- net +5V: now also R?.1
- net 36V: now also TP3.1
- net EN: now also R?.2; no longer R?.1
- net GND: no longer R?.2
Other:
- moved on the sheet: R?
Changed lines of the file:
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@@
   (junction (at 134.62 82.55) (diameter 0) (color 0 0 0 0)
   )
+  (junction (at 179.07 82.55) (diameter 0) (color 0 0 0 0)
+  )
+  (junction (at 106.68 87.63) (diameter 0) (color 0 0 0 0)
+  )
   (junction (at 96.52 82.55) (diameter 0) (color 0 0 0 0)
   )
@@
   (junction (at 185.42 82.55) (diameter 0) (color 0 0 0 0)
   )
-  (junction (at 106.68 93.98) (diameter 0) (color 0 0 0 0)
-  )
   (wire (pts (xy 147.32 95.25) (xy 147.32 97.79))
     (stroke (width 0) (type default))
@@
     (stroke (width 0) (type default))
   )
-  (wire (pts (xy 96.52 80.01) (xy 96.52 82.55))
-    (stroke (width 0) (type default))
-  )
-  (wire (pts (xy 171.45 82.55) (xy 185.42 82.55))
+  (wire (pts (xy 96.52 69.85) (xy 96.52 82.55))
+    (stroke (width 0) (type default))
+  )
+  (wire (pts (xy 171.45 82.55) (xy 179.07 82.55))
     (stroke (width 0) (type default))
   )
@@
     (stroke (width 0) (type default))
   )
-  (wire (pts (xy 106.68 93.98) (xy 106.68 96.52))
-    (stroke (width 0) (type default))
-  )
   (wire (pts (xy 171.45 92.71) (xy 171.45 95.25))
     (stroke (width 0) (type default))
   )
+  (wire (pts (xy 179.07 80.01) (xy 179.07 82.55))
+    (stroke (width 0) (type default))
+  )
   (wire (pts (xy 132.08 87.63) (xy 135.89 87.63))
     (stroke (width 0) (type default))
@@
     (stroke (width 0) (type default))
   )
+  (wire (pts (xy 106.68 80.01) (xy 106.68 87.63))
+    (stroke (width 0) (type default))
+  )
   (wire (pts (xy 185.42 92.71) (xy 185.42 95.25))
     (stroke (width 0) (type default))
@@
     (stroke (width 0) (type default))
   )
+  (wire (pts (xy 106.68 69.85) (xy 106.68 72.39))
+    (stroke (width 0) (type default))
+  )
   (wire (pts (xy 147.32 107.95) (xy 147.32 110.49))
     (stroke (width 0) (type default))
@@
     (stroke (width 0) (type default))
   )
-  (wire (pts (xy 106.68 104.14) (xy 106.68 106.68))
+  (wire (pts (xy 179.07 82.55) (xy 185.42 82.55))
     (stroke (width 0) (type default))
   )
@@
       (effects (font (size 1.27 1.27)) hide)
     )
+    (property "LCSC" "C122547" (at 147.32 104.14 0)
+      (effects (font (size 1.27 1.27)) hide)
+    )
     (pin "1")
     (pin "2")
@@
       (effects (font (size 1.27 1.27)) hide)
     )
+    (property "LCSC" "C1683" (at 158.75 88.9 0)
+      (effects (font (size 1.27 1.27)) hide)
+    )
     (pin "1")
     (pin "2")
@@
     )
   )
-  (symbol (lib_id "Device:R") (at 106.68 100.33 0) (unit 1)
-    (in_bom yes) (on_board yes) (dnp no) (fields_autoplaced)
-    (property "Reference" "R?" (at 109.22 99.695 0)
-      (effects (font (size 1.27 1.27)) (justify left))
-    )
-    (property "Value" "47K" (at 109.22 102.235 0)
-      (effects (font (size 1.27 1.27)) (justify left))
-    )
-    (property "Footprint" "Resistor_SMD:R_0402_1005Metric" (at 104.902 100.33 90)
-      (effects (font (size 1.27 1.27)) hide)
-    )
-    (property "Datasheet" "~" (at 106.68 100.33 0)
+  (symbol (lib_id "Device:R") (at 106.68 76.2 0) (unit 1)
+    (in_bom yes) (on_board yes) (dnp no) (fields_autoplaced)
+    (property "Reference" "R?" (at 109.22 75.565 0)
+      (effects (font (size 1.27 1.27)) (justify left))
+    )
+    (property "Value" "100K" (at 109.22 78.105 0)
+      (effects (font (size 1.27 1.27)) (justify left))
+    )
+    (property "Footprint" "Resistor_SMD:R_0402_1005Metric" (at 104.902 76.2 90)
+      (effects (font (size 1.27 1.27)) hide)
+    )
+    (property "Datasheet" "~" (at 106.68 76.2 0)
+      (effects (font (size 1.27 1.27)) hide)
+    )
+    (property "LCSC" "C25741" (at 106.68 76.2 0)
       (effects (font (size 1.27 1.27)) hide)
     )
@@
       (effects (font (size 1.27 1.27)) hide)
     )
+    (property "LCSC" "C2045998" (at 124.46 69.85 90)
+      (effects (font (size 1.27 1.27)) hide)
+    )
     (pin "1")
     (pin "2")
@@
       (effects (font (size 1.27 1.27)))
     )
+    (property "LCSC" "C23630" (at 185.42 88.9 0)
+      (effects (font (size 1.27 1.27)) hide)
+    )
     (pin "1")
     (pin "2")
@@
         (path "/3a5f1087-1abe-4575-9313-bd86a5e03366/1f5aaf38-830e-4ce3-b87a-a54930c92dff"
           (reference "#PWR054") (unit 1)
+        )
+      )
+    )
+  )
+  (symbol (lib_id "power:+5V") (at 106.68 69.85 0) (unit 1)
+    (in_bom yes) (on_board yes) (dnp no) (fields_autoplaced)
+    (property "Reference" "#PWR02" (at 106.68 73.66 0)
+      (effects (font (size 1.27 1.27)) hide)
+    )
+    (property "Value" "+5V" (at 106.68 66.04 0)
+      (effects (font (size 1.27 1.27)))
+    )
+    (property "Footprint" "" (at 106.68 69.85 0)
+      (effects (font (size 1.27 1.27)) hide)
+    )
+    (property "Datasheet" "" (at 106.68 69.85 0)
+      (effects (font (size 1.27 1.27)) hide)
+    )
+    (pin "1")
+    (instances
+      (project "emonHP"
+        (path "/3a5f1087-1abe-4575-9313-bd86a5e03366/1f5aaf38-830e-4ce3-b87a-a54930c92dff"
+          (reference "#PWR02") (unit 1)
         )
       )
@@
     )
     (property "Mouser" "926-LM2733XMFX/NOPB" (at 124.46 85.09 0)
+      (effects (font (size 1.27 1.27)) hide)
+    )
+    (property "LCSC" "C78226" (at 124.46 85.09 0)
       (effects (font (size 1.27 1.27)) hide)
     )
@@
     )
   )
+  (symbol (lib_id "Connector:TestPoint") (at 179.07 80.01 0) (unit 1)
+    (in_bom no) (on_board yes) (dnp no) (fields_autoplaced)
+    (property "Reference" "TP3" (at 181.61 76.073 0)
+      (effects (font (size 1.27 1.27)) (justify left))
+    )
+    (property "Value" "TestPoint" (at 181.61 78.613 0)
+      (effects (font (size 1.27 1.27)) (justify left))
+    )
+    (property "Footprint" "TestPoint:TestPoint_Pad_D1.0mm" (at 184.15 80.01 0)
+      (effects (font (size 1.27 1.27)) hide)
+    )
+    (property "Datasheet" "~" (at 184.15 80.01 0)
+      (effects (font (size 1.27 1.27)) hide)
+    )
+    (pin "1")
+    (instances
+      (project "emonHP"
+        (path "/3a5f1087-1abe-4575-9313-bd86a5e03366/1f5aaf38-830e-4ce3-b87a-a54930c92dff"
+          (reference "TP3") (unit 1)
+        )
+      )
+    )
+  )
   (symbol (lib_id "Device:C") (at 171.45 88.9 0) (unit 1)
     (in_bom yes) (on_board yes) (dnp no)
@@
       (effects (font (size 1.27 1.27)))
     )
+    (property "LCSC" "C23630" (at 171.45 88.9 0)
+      (effects (font (size 1.27 1.27)) hide)
+    )
     (pin "1")
     (pin "2")
@@
       (effects (font (size 1.27 1.27)))
     )
-    (property "Value" "MBR0550" (at 141.2875 80.01 0)
+    (property "Value" "MBR0580" (at 141.2875 80.01 0)
       (effects (font (size 1.27 1.27)))
     )
@@
       (effects (font (size 1.27 1.27)) hide)
     )
+    (property "LCSC" "C177047" (at 140.97 82.55 0)
+      (effects (font (size 1.27 1.27)) hide)
+    )
     (pin "1")
     (pin "2")
@@
     )
   )
-  (symbol (lib_id "power:GND") (at 106.68 106.68 0) (unit 1)
-    (in_bom yes) (on_board yes) (dnp no) (fields_autoplaced)
-    (property "Reference" "#PWR?" (at 106.68 113.03 0)
-      (effects (font (size 1.27 1.27)) hide)
-    )
-    (property "Value" "GND" (at 106.68 111.76 0)
-      (effects (font (size 1.27 1.27)))
-    )
-    (property "Footprint" "" (at 106.68 106.68 0)
-      (effects (font (size 1.27 1.27)) hide)
-    )
-    (property "Datasheet" "" (at 106.68 106.68 0)
-      (effects (font (size 1.27 1.27)) hide)
-    )
-    (pin "1")
-    (instances
-      (project "mbus-reader-proto"
-        (path "/36d146b0-f348-4341-a935-471af0e684a6"
-          (reference "#PWR?") (unit 1)
-        )
-        (path "/36d146b0-f348-4341-a935-471af0e684a6/d9d13df7-ec5a-4d9a-8998-14ae0ed59560"
-          (reference "#PWR?") (unit 1)
-        )
-      )
-      (project "emonHP"
-        (path "/3a5f1087-1abe-4575-9313-bd86a5e03366/1f5aaf38-830e-4ce3-b87a-a54930c92dff"
-          (reference "#PWR052") (unit 1)
-        )
-      )
-    )
-  )
   (symbol (lib_id "Device:C") (at 96.52 88.9 0) (unit 1)
     (in_bom yes) (on_board yes) (dnp no) (fields_autoplaced)
@@
       (effects (font (size 1.27 1.27)) hide)
     )
+    (property "LCSC" "C23630" (at 96.52 88.9 0)
+      (effects (font (size 1.27 1.27)) hide)
+    )
     (pin "1")
     (pin "2")
@@
       (effects (font (size 1.27 1.27)) hide)
     )
+    (property "LCSC" "C25557" (at 147.32 88.9 0)
+      (effects (font (size 1.27 1.27)) hide)
+    )
     (pin "1")
     (pin "2")
@@
     )
   )
-  (symbol (lib_id "power:+5V") (at 96.52 80.01 0) (unit 1)
-    (in_bom yes) (on_board yes) (dnp no) (fields_autoplaced)
-    (property "Reference" "#PWR?" (at 96.52 83.82 0)
-      (effects (font (size 1.27 1.27)) hide)
-    )
-    (property "Value" "+5V" (at 96.52 76.2 0)
-      (effects (font (size 1.27 1.27)))
-    )
-    (property "Footprint" "" (at 96.52 80.01 0)
-      (effects (font (size 1.27 1.27)) hide)
-    )
-    (property "Datasheet" "" (at 96.52 80.01 0)
-      (effects (font (size 1.27 1.27)) hide)
-    )
+  (symbol (lib_id "power:+5V") (at 96.52 69.85 0) (unit 1)
+    (in_bom yes) (on_board yes) (dnp no) (fields_autoplaced)
+    (property "Reference" "#PWR?" (at 96.52 73.66 0)
+      (effects (font (size 1.27 1.27)) hide)
+    )
+    (property "Value" "+5V" (at 96.52 66.04 0)
+      (effects (font (size 1.27 1.27)))
+    )
+    (property "Footprint" "" (at 96.52 69.85 0)
+      (effects (font (size 1.27 1.27)) hide)
+    )
+    (property "Datasheet" "" (at 96.52 69.85 0)
+      (effects (font (size 1.27 1.27)) hide)
+    )
